File: ArduF405_Hardware.kicad_pcb (KiCad board)
At the start: 2 copper layers, 40.5 x 40.5 mm, 90 parts, among them J1 USB_C_Receptacle_USB2.0, J10 Micro_SD_Card, J3 GPS, J6 ESC, J7 Upper computer connector, Q1 AP40P05, U1 MP9943GQ-Z, U2 RT9013-33GB, U3 RT9013-33GB, U4 STM32F405RGTx, U5 BMI270, U6 AT7456E, U7 W25Q128JVS, U8 SPL06, Y1 YXC 0T252016MJBA4SL, Y2 YXC_XG1EL89CSI-111YLC-27M 27M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

Commit message: 完成原理图绘制
Parts:
- added J11: USART_3, NxtPX4:01x04_MP_sh1.0_Hori, F.Cu at (145.5, -27.7)
- added J12: UART_5, NxtPX4:01x04_MP_sh1.0_Hori, F.Cu at (145.5, -20.8)
- added J8: ESC_2, NxtPX4:01x08_MP_sh1.0_Hori, F.Cu at (155.5, -34.6)
- added J9: USART_1, NxtPX4:01x04_MP_sh1.0_Hori, F.Cu at (145.5, -34.6)
Connections:
- U6 pad 29: GND -> (no net)
Other:
- board outline removed

Commit message: 完成PCB板设计
Parts:
- removed J11: USART_3, NxtPX4:01x04_MP_sh1.0_Hori
- added C19: 10uF(0603 35V 20%), Capacitor_SMD:C_0603_1608Metric, B.Cu at (118.4, 119.0)
- added C20: 1uF(0402 35V 10%), Capacitor_SMD:C_0402_1005Metric, B.Cu at (115.8, 117.8)
- added C21: 100nF(0603 10V 10%), Capacitor_SMD:C_0603_1608Metric, B.Cu at (115.2, 122.2)
- added C22: 100nF(0603 25V 10%), Capacitor_SMD:C_0603_1608Metric, B.Cu at (118.4, 117.3)
- added C44: 22uF(0603 16V), Capacitor_SMD:C_0603_1608Metric, B.Cu at (118.4, 114.1)
- added C45: 22uF(0603 16V), Capacitor_SMD:C_0603_1608Metric, B.Cu at (118.4, 115.8)
- added D10: LED_blue, LED_SMD:LED_0603_1608Metric, F.Cu at (103.9, 102.1)
- added D8: LED_Red, LED_SMD:LED_0603_1608Metric, F.Cu at (103.9, 98.8)
- added D9: LED_blue, LED_SMD:LED_0603_1608Metric, F.Cu at (103.9, 100.5)
- added J: pad, Library:1p_1.5mm_Pad, F.Cu at (94.6, 121.8)
- added J: pad, Library:1p_1.5mm_Pad, F.Cu at (94.6, 125.8)
- added J: pad, Library:1p_1.5mm_Pad, F.Cu at (94.6, 123.8)
- added J: pad, Library:1p_1.5mm_Pad, F.Cu at (94.6, 117.8)
- added J: pad, Library:1p_1.5mm_Pad, F.Cu at (94.6, 119.8)
- added J2: CAM, NxtPX4:01x03_MP_sh1.0_Hori, F.Cu at (109.8, 99.6)
- added J4: VTX, NxtPX4:01x05_MP_sh1.0_Hori, F.Cu at (118.7, 99.6)
- added J5: DJI O4, NxtPX4:1x06-1MP_P1.00mm_Horizontal, B.Cu at (110.6, 99.5)
- added L2: 10uH(0420)(78438357100), NxtPX4:Inductor_0420, B.Cu at (123.7, 114.5)
- added R10: 20R(0603 25V), Resistor_SMD:R_0603_1608Metric, B.Cu at (118.4, 123.9)
- added R12: 51kR(0603 25V), Resistor_SMD:R_0603_1608Metric, B.Cu at (118.4, 120.6)
- added R18: 3.6kR(0603 25V), Resistor_SMD:R_0603_1608Metric, B.Cu at (115.2, 123.9)
- added R19: 41.2kR(0603 25V), Resistor_SMD:R_0603_1608Metric, B.Cu at (118.4, 122.2)
- added R20: 3.6kR(0603 25V), Resistor_SMD:R_0603_1608Metric, F.Cu at (100.6, 98.9)
- added R21: 3.6kR(0603 25V), Resistor_SMD:R_0603_1608Metric, F.Cu at (100.6, 100.5)
- added R22: 3.6kR(0603 25V), Resistor_SMD:R_0603_1608Metric, F.Cu at (100.6, 102.1)
- added R35: 10kR(0603), Resistor_SMD:R_0603_1608Metric, B.Cu at (124.8, 137.2)
- added R36: 10kR(0603), Resistor_SMD:R_0603_1608Metric, B.Cu at (124.9, 138.8)
- added R5: 1MR(0402 50V), Resistor_SMD:R_0402_1005Metric, B.Cu at (115.8, 119.0)
- added R6: 100kR(0603 25V), Resistor_SMD:R_0603_1608Metric, B.Cu at (115.2, 120.6)
- added U19: SN74LVC1G86DCKR, NxtPX4:DCK5, F.Cu at (124.7, 137.8)
- added U9: MP9943GQ-Z, NxtPX4:MP9943GQ-Z, B.Cu at (111.2, 122.4)
- C1, C11, C14, C15, C2, C32, C33, C34, C35, C36, C38, C39, C4, C40, C5, C6, C9, D1, D2, D3, D4, D5, D7, J10, J3, J8, J9, L1, R14, R15, R29, R3, R30, R4, TP1, U1, U5: moved to B.Cu
- H1, H2, H3, H4: footprint MountingHole:MountingHole_3mm_Pad -> MountingHole:MountingHole_4.3mm_M4_DIN965_Pad
- J12: value UART_5 -> UART_4; moved to B.Cu
- J7: value Upper computer connector -> Upper computer connector/RC input
- moved C2 206.7 mm to (114.6, 130.4)
- moved C7 206.1 mm to (117.5, 131.2)
- moved R14 204.7 mm to (111.4, 132.1), turned to 180 degrees
- moved R4 204.1 mm to (117.8, 130.4), turned to 180 degrees
- moved R8 203.3 mm to (118.4, 134.4)
- moved R7 203.1 mm to (115.2, 132.8)
- moved C17 201.8 mm to (117.2, 129.2), turned to 180 degrees
- moved R15 200.8 mm to (111.4, 130.5)
- moved C4 200.2 mm to (115.4, 135.7), turned to 180 degrees
- moved R9 199.5 mm to (118.4, 132.8)
- moved C14 198.3 mm to (107.4, 131.8), turned to 90 degrees
- moved C23 195.6 mm to (110.9, 127.5)
- moved C5 194.7 mm to (106.3, 133.8), turned to -90 degrees
- moved C15 194.5 mm to (108.5, 129.8), turned to -90 degrees
- moved C24 194.4 mm to (114.1, 127.5), turned to 180 degrees
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Connections:
- net System_5V renamed Net-(D7-A)
- H1 pad 1: GNDD -> GND
- H2 pad 1: GNDD -> GND
- H3 pad 1: GNDD -> GND
- H4 pad 1: GNDD -> GND
- J12 pad 3: /UART5_TX -> /UART4_TX
- J12 pad 4: /UART5_RX -> /UART4_RX
- J6 pad 6: unconnected-(J6-Pin_6-Pad6) -> /USART3_RX
- J7 pad 4: /TIM9_CH2 -> /SBUS
- J8 pad 6: unconnected-(J8-Pin_6-Pad6) -> /USART3_RX
- U4 pad 26: unconnected-(U4-PB0-Pad26) -> /SBUS_INV
- U4 pad 46: unconnected-(U4-PA13-Pad46) -> /LED_0
- U4 pad 49: unconnected-(U4-PA14-Pad49) -> /LED_1
- U6 pad 29: (no net) -> GND
Routing:
- net Core_3V3: track 0.00 -> 218.6 mm, vias 0 -> 14
- net System_4V5: track 0.00 -> 128.6 mm, vias 0 -> 8
- net /TIM11_CH1: track 0.00 -> 64.5 mm
- net /SBUS: track 0.00 -> 56.8 mm, vias 0 -> 1
- net /I2C1_SCL: track 0.00 -> 55.5 mm, vias 0 -> 2
- net /I2C1_SDA: track 0.00 -> 54.9 mm, vias 0 -> 2
- net CAM_10V: track 0.00 -> 54.5 mm, vias 0 -> 4
- net /USART3_RX: track 0.00 -> 52.4 mm, vias 0 -> 3
- net /UART5_RX: track 0.00 -> 52.2 mm, vias 0 -> 1
- net /TIM2_CH2: track 0.00 -> 49.7 mm, vias 0 -> 1
- net /TIM2_CH1: track 0.00 -> 49.1 mm, vias 0 -> 1
- net /UART5_TX: track 0.00 -> 48.2 mm, vias 0 -> 1
- net /TIM9_CH2: track 0.00 -> 44.7 mm, vias 0 -> 2
- net VCC_24V: track 0.00 -> 38.9 mm, vias 0 -> 4
- net /USART2_TX: track 0.00 -> 36.9 mm, vias 0 -> 2
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- added copper zone on In2.Cu, net CAM_10V
- added copper zone on In2.Cu, net Core_3V3
- added copper zone on B.Cu, net GND
- added copper zone on F.Cu, net GND
- added copper zone on In1.Cu, net GND
- added copper zone on In2.Cu, net Periph_3V3
- added copper zone on In2.Cu, net System_4V5
- added copper zone on F.Cu, net VCC_24V
- added copper zone on F.Cu, net VCC_BAT
Other:
- board outline added: 35.8 x 45.8 mm
- copper layers 2 -> 4

Commit message: 添加丝印
Parts:
- added G***: LOGO, 文档:ArduPilot_logo, B.Cu at (93.8, 119.3)
- moved J 9.02 mm to (94.0, 112.8)
- moved J 5.53 mm to (94.0, 120.3)
- moved J 4.54 mm to (94.0, 115.3)
- moved J 1.17 mm to (94.0, 122.8)
- moved J 0.60 mm to (94.0, 117.8)
Routing:
- net System_4V5: track 128.6 -> 123.5 mm
Other:
- board text added: "4V5"
- board text added: "CAM"
- board text added: "DJI"
- board text added: "G"
- board text added: "GPS"
- board text added: "PR"
- board text added: "RC"
- board text added: "SCL"
- board text added: "SDA"
- board text added: "UART1"
- board text added: "UART4"
- board text added: "VTX"
